File: PCBs/ninjaCam/ninjaCam.kicad_sch (KiCad schematic)
At the start: 15 parts, among them J1 DVI-HX-107DIP

Commit message: connected pin8 of VGa to GND was NC before
on hat/fpga also connected to gnd
Connections:
- net GND: now also J1.8
Changed lines of the file:
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@@
   (junction (at 205.105 40.005) (diameter 0) (color 0 0 0 0)
+  )
+  (junction (at 147.32 78.74) (diameter 0) (color 0 0 0 0)
   )
   (junction (at 205.105 65.405) (diameter 0) (color 0 0 0 0)
@@
     (stroke (width 0) (type default) (color 0 0 0 0))
   )
+  (wire (pts (xy 147.32 78.74) (xy 147.32 81.28))
+    (stroke (width 0) (type default) (color 0 0 0 0))
+  )
